File: STM.sch (KiCad schematic (older format))
At the start: 21 parts

Commit message: added RPi Regulator added ref.des.-prefixes to all schematic sheets
Other:
- note added: "Ref: 7x & 8x"
Changed lines of the file:
@@
 	2450 1300 2650 1300
 Connection ~ 2650 1300
+Text Notes 10025 6525 0    118  ~ 0
+Ref: 7x & 8x
 $EndSCHEMATC
