File: Logic_Hedgehog.sch (KiCad schematic (older format))
At the start: 12 parts

Commit message: moved stuff from other sheet to Logic sheet cleanup added connections schematic nearly finished
Parts:
- added C? (x4): 1µ, symbol C
- added C? (x2): 22p, symbol C
- added C? (x3): 2µ2, symbol C
- added C? (x7): 100n, symbol C
- added C? (x2): 10µ, symbol C
- added C?: 0µ47, symbol C
- added D? (x7): 3V3, symbol D_Zener
- added D? (x2): LED, symbol LED
- added J?: SPI_EXT_0_0, symbol CONN_01X06
- added J?: SPI_EXT_0_1, symbol CONN_01X06
- added J?: I2C_EXT_0, symbol CONN_01X04
- added J?: I2C_EXT_1, symbol CONN_01X04
- added J?: UART_EXT_1, symbol CONN_01X04
- added J? (x2): MOTORS, symbol CONN_01X04
- added J?: SPI_EXT_1, symbol CONN_01X06
- added L?: 39n, symbol L
- added R? (x2): R, symbol R
- added R?: 22R, symbol R
- added R?: 0R, symbol R
- added R? (x2): 1k8, symbol R
- added R? (x2): 330R, symbol R
- added U?: STM32F401VBT6, symbol STM32F401VBT6
- added U? (x2): DRV8835, hedgehog_footprints:WSON12, symbol DRV8835
- added U?: IMU_ICM-20689, symbol IMU_ICM-20689
- added Y?: Crystal, symbol Crystal
- R? (x2): value 330 -> 330R
- U?: value Piezo-Buzzer -> Buzzer
Connections:
- net +3V3: now also C?.1, C?.1, C?.2, C?.2, C?.2, C?.2, C?.2, C?.2, C?.2, J?.2 (P2), J?.2 (P2), J?.2 (P2), J?.2 (P2), J?.2 (P2), J?.2 (P2), L?.1, R?.2, R?.2, R?.2, U?.100 (VDD), U?.11 (VDD), U?.12 (VCC), U?.12 (VCC), U?.19 (VDD), U?.28 (VDD), U?.50 (VDD), U?.6 (VBAT), U?.75 (VDD), U?.8 (VDDIO)
- net +5V: now also C?.1, C?.1, C?.2, U?.1 (VM), U?.1 (VM)
- net EN_PWR_IN: now also U?.57 (PD10)
- net EN_Reg_MS: now also U?.56 (PD9)
- net EN_Reg_RPi: now also U?.55 (PD8)
- net GND: now also U?.6 (GND), C?.1, C?.1, C?.1, C?.1, C?.1, C?.1, C?.1, C?.1, C?.1, C?.1, C?.1, C?.1, C?.2, C?.2, C?.2, C?.2, C?.2, C?.2, C?.2, D?.1 (K), D?.1 (K), D?.2 (A), D?.2 (A), D?.2 (A), D?.2 (A), D?.2 (A), D?.2 (A), D?.2 (A), J?.1 (P1), J?.1 (P1), J?.1 (P1), J?.1 (P1), J?.1 (P1), J?.1 (P1), R?.2, U?.10 (GND), U?.11 (FSYNC), U?.18 (GND), U?.20 (VSSA/VREF-), U?.27 (GND), U?.49 (GND), U?.6 (GND), U?.6 (GND), U?.74 (GND), U?.99 (GND)
- net POWER_IN_SENSE: now also U?.36 (PB1)
- net PWR_BUTTON_STATE: now also U?.58 (PD11)
- net STM_NJTRST: now reaches U?.11 (GPIO17)
- net STM_NJTRST: now also U?.90 (PB4)
- net STM_JTDO_SWO: now reaches U?.13 (GPIO27)
- net STM_JTDO_SWO: now also U?.89 (PB3)
- net STM_JTDI: now reaches U?.15 (GPIO22)
- net STM_JTDI: now also U?.77 (PA15)
- net SPI_EXT_0_MOSI: now reaches U?.19 (GPIO10)
- net SPI_EXT_0_MOSI: now also D?.1 (K), J?.5 (P5), J?.5 (P5)
- net SPI_EXT_0_MISO: now reaches U?.21 (GPIO09)
- net SPI_EXT_0_MISO: now also D?.1 (K), J?.6 (P6), J?.6 (P6)
- net SPI_EXT_0_SCK: now reaches U?.23 (GPIO11)
- net SPI_EXT_0_SCK: now also D?.1 (K), J?.4 (P4), J?.4 (P4)
- net SPI_EXT_0_NSS0: now reaches U?.24 (GPIO08)
- net SPI_EXT_0_NSS0: now also D?.1 (K), J?.3 (P3)
- net SPI_EXT_0_NSS1: now reaches U?.26 (GPIO07)
- net SPI_EXT_0_NSS1: now also D?.1 (K), J?.3 (P3)
- net STM_NRST: now reaches U?.29 (GPIO05)
- net STM_NRST: now also R?.1, U?.14 (NRST)
- net I2C_EXT_0_SDA: now reaches U?.3 (GPIO02)
- net I2C_EXT_0_SDA: now also D?.1 (K), J?.4 (P4)
- net STM_BOOT0: now reaches U?.31 (GPIO06)
- net STM_BOOT0: now also R?.1, U?.94 (BOOT0)
- net STM_JTCK_SWCLK: now reaches U?.33 (GPIO13)
- net STM_JTCK_SWCLK: now also U?.76 (PA14)
- net STM_JTMS_SWDIO: now reaches U?.35 (GPIO19)
- net STM_JTMS_SWDIO: now also U?.72 (PA13)
- net LED_3: now reaches U?.38 (GPIO20)
- net LED_3: now also R?.1
- net LED_4: now reaches U?.40 (GPIO21)
- net LED_4: now also R?.1
- net I2C_EXT_0_SCL: now reaches U?.5 (GPIO03)
- net I2C_EXT_0_SCL: now also D?.1 (K), J?.3 (P3)
- net BUZZER_N: now reaches U?.2
- net BUZZER_N: now also U?.39 (PE8)
- net PA0 renamed BUZZER_P
- net BUZZER_P: now also U?.40 (PE9)
- net PA1 renamed ANALOG_0
- net ANALOG_0: now also U?.24 (PA1), U?.81 (PD0)
- net PA10 renamed RPi_UART_TxD
- net RPi_UART_TxD: now also U?.69 (PA10)
- net PA11 renamed LED_1
- net LED_1: now also U?.95 (PB8)
- net PA12 renamed LED_2
- net LED_2: now also U?.96 (PB9)
- net PA2 renamed ANALOG_1
- net ANALOG_1: now also U?.25 (PA2), U?.82 (PD1)
- net PA3 renamed ANALOG_2
- net ANALOG_2: now also U?.26 (PA3), U?.83 (PD2)
- net PA4 renamed ANALOG_3
- net ANALOG_3: now also U?.29 (PA4), U?.84 (PD3)
- net PA5 renamed ANALOG_4
- net ANALOG_4: now also U?.30 (PA5), U?.85 (PD4)
- net PA6 renamed ANALOG_5
- net ANALOG_5: now also U?.31 (PA6), U?.86 (PD5)
- net PA7 renamed ANALOG_6
- net ANALOG_6: now also U?.32 (PA7), U?.87 (PD6)
- net PA9 renamed RPi_UART_RxD
- net RPi_UART_RxD: now also U?.68 (PA9)
- net PB0 renamed ANALOG_7
- net ANALOG_7: now also U?.35 (PB0)
- net PD12 renamed SERVO_0
- net SERVO_0: now also U?.59 (PD12)
- net PD13 renamed SERVO_1
- net SERVO_1: now also U?.60 (PD13)
- net PD14 renamed SERVO_2
- net SERVO_2: now also U?.61 (PD14)
- net PD15 renamed SERVO_3
- net SERVO_3: now also U?.62 (PD15)
- net PE10 renamed DIGITAL_2
- net DIGITAL_2: now also U?.41 (PE10)
- net PE11 renamed DIGITAL_3
- net DIGITAL_3: now also U?.42 (PE11)
- net PE12 renamed DIGITAL_4
- net DIGITAL_4: now also U?.43 (PE12)
- net PE13 renamed DIGITAL_5
- net DIGITAL_5: now also U?.44 (PE13)
- net PE14 renamed DIGITAL_6
- net DIGITAL_6: now also U?.45 (PE14)
- net PE15 renamed DIGITAL_7
- net DIGITAL_7: now also U?.46 (PE15)
- net PE8 renamed DIGITAL_0
- net DIGITAL_0: now also U?.97 (PE0)
- net PE9 renamed DIGITAL_1
- net DIGITAL_1: now also U?.98 (PE1)
- new net: R?.1, U?.12 (PH0-OSC_IN)
- new net: R?.1, U?.13 (PH1_OSC_OUT)
- new net: C?.2, U?.48 (VCAP_1)
- new net: C?.2, U?.73 (VCAP_2)
- new net: C?.1, R?.2, Y?.1
- new net: C?.1, R?.2, Y?.2
- new net: J?.1 (P1), U?.2 (AOUT1)
- new net: J?.1 (P1), U?.3 (AOUT2)
- new net: J?.2 (P2), U?.4 (BOUT1)
- new net: J?.2 (P2), U?.5 (BOUT2)
- new net: J?.3 (P3), U?.2 (AOUT1)
- new net: J?.3 (P3), U?.3 (AOUT2)
- new net: J?.4 (P4), U?.4 (BOUT1)
- new net: J?.4 (P4), U?.5 (BOUT2)
- new net: D?.2 (A), R?.2 (x2)
- new net: C?.2, U?.10 (REGOUT)
- new net I2C_EXT_1_SCL: J?.3 (P3), R?.1, U?.92 (PB6)
- new net I2C_EXT_1_SDA: J?.4 (P4), R?.1, U?.93 (PB7)
- new net IMU_INT: U?.12 (INT), U?.2 (PE3)
- new net IMU_MISO: U?.4 (PE5), U?.9 (AD0/SD0)
- new net IMU_MOSI: U?.24 (SDA/SDI), U?.5 (PE6)
- new net IMU_NCS: U?.22 (nCS), U?.3 (PE4)
- new net IMU_SCK: U?.1 (PE2), U?.23 (SCL/SCLK)
- new net MOTOR_01: U?.11 (MODE), U?.15 (PC0)
- new net MOTOR_0_A: U?.10 (AIN1/APHASE), U?.16 (PC1)
- new net MOTOR_0_B: U?.63 (PC6), U?.9 (AIN2/AENBL)
- new net MOTOR_1_A: U?.17 (PC2), U?.8 (BIN1/BPHASE)
- new net MOTOR_1_B: U?.64 (PC7), U?.7 (BIN2/BENBL)
- new net MOTOR_23: U?.11 (MODE), U?.34 (PC5)
- new net MOTOR_2_A: U?.10 (AIN1/APHASE), U?.18 (PC3)
- new net MOTOR_2_B: U?.65 (PC8), U?.9 (AIN2/AENBL)
- new net MOTOR_3_A: U?.33 (PC4), U?.8 (BIN1/BPHASE)
- new net MOTOR_3_B: U?.66 (PC9), U?.7 (BIN2/BENBL)
- new net SPI_EXT_1_MISO: J?.6 (P6), U?.53 (PB14)
- new net SPI_EXT_1_MOSI: J?.5 (P5), U?.54 (PB15)
- new net SPI_EXT_1_NSS: J?.3 (P3), U?.51 (PB12)
- new net SPI_EXT_1_SCK: J?.4 (P4), U?.52 (PB13)
- new net UART_EXT_1_RxD: J?.4 (P4), U?.71 (PA12)
- new net UART_EXT_1_TxD: J?.3 (P3), U?.70 (PA11)
- new net VDDA: C?.1, C?.2, L?.2, U?.13 (VDD), U?.21 (VREF+), U?.22 (VDDA)
- no-connect marks 0 -> 12
Other:
- note added: "Analog Inputs"
- note added: "Digital Inputs"
- note added: "Inerfaces + RPi Protection"
- note added: "LEDs"
- note added: "Motor Drivers"
- note added: "Ref: 4x, 5x"
- note added: "SPI4"
- note added: "Servos"
- note added: "TIM1_CH1"
- note added: "UART6"
- note added: "pi resets stm during boot/when off?\nhigh on reset line when pi off -> bad for pi?"
- note removed: "ADC"
- note removed: "Analog Input"
- note removed: "Digital Input"
- note removed: "INT FOR I2C ?"
- note removed: "JTCK-SWCLK"
- note removed: "JTDI"
- note removed: "JTMS(SWDIO)"
- note removed: "MISO"
- note removed: "MOSI"
- note removed: "Motor"
- note removed: "NSS"
- note removed: "Piezo-Buzzer"
- note removed: "Problem: 2 net names"
- note removed: "RX"
- note removed: "Ref: 4x"
- note removed: "SCK"
- note removed: "SPI1"
- note removed: "Servo"
- note removed: "TODO: Timer1"
- note removed: "TX"
- moved on the sheet: D?, J?, R?, U?

Commit message: changed zener values added comments
Parts:
- D? (x7): value 3V3 -> 3V6
Other:
- note added: "Microcontroller"
- note added: "Raspberry Pi 3"
- note added: "protection ok?"
- moved on the sheet: C?, J?, U?

Commit message: Added Symbolnames
Parts:
- gave numbers to parts that had none: 61
Other:
- moved on the sheet: U44
