File: Logic.sch (KiCad schematic (older format))
At the start: 69 parts, among them J40 RaspberryPi3, J41 UART_EXT_1, J42 I2C_EXT_0, J43 I2C_EXT_0_EXP, J44 I2C_EXT_1, J45 SPI_EXT_0_0, J46 SPI_EXT_0_1, J47 SPI_EXT_1, J48 I/O_0-7, J49 I/O_8-15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

Commit message: lots of changes: regulator layout improved bom minimized inner top layer completely gnd UB single pole pullups for use without pi swiched to new kicad version and fp lib motor and servo netanmes fixed added input filtering
Parts:
- removed JP1: Jumper, hedgehog_footprints:Pin_Header_Straight_1x02_Pitch2.54mm, symbol Device:Jumper
- added JP1: UB, Connector_Pin:Pin_D1.0mm_L10.0mm, symbol Connector_Generic:Conn_01x01
- added R52, R53, R54: 1k6, Resistor_SMD:R_0603_1608Metric, symbol Device:R
- C40, C41, C42, C43, C44, C45, C46, C47, C48, C49, C50, C51, C61, C62, C63: footprint Capacitors_SMD:C_0603 -> Capacitor_SMD:C_0603_1608Metric
- C52: renamed from C54; footprint Capacitors_SMD:C_0603 -> Capacitor_SMD:C_0603_1608Metric
- C53: renamed from C55; footprint Capacitors_SMD:C_0603 -> Capacitor_SMD:C_0603_1608Metric
- C54: renamed from C52; footprint Capacitors_SMD:C_0603 -> Capacitor_SMD:C_0603_1608Metric
- C55: renamed from C53; footprint Capacitors_SMD:C_0603 -> Capacitor_SMD:C_0603_1608Metric
- D40, D41, D42, D43, D51: footprint LEDs:LED_0805 -> LED_SMD:LED_0805_2012Metric
- D44, D45, D46, D47, D48, D49, D50: footprint hedgehog_footprints:SOD323F -> Diode_SMD:D_SOD-323F
- L40: footprint Inductors_SMD:L_0603 -> Inductor_SMD:L_0603_1608Metric
- R40, R41, R42, R43, R44, R45, R46, R47, R48, R49, R50, R51: footprint Resistors_SMD:R_0603 -> Resistor_SMD:R_0603_1608Metric
- U40: footprint hedgehog_footprints:LQFP_100 -> Package_QFP:LQFP-100_14x14mm_P0.5mm
- U41: footprint Housings_SSOP:VSSOP-8_2.3x2mm_Pitch0.5mm -> Package_SO:VSSOP-8_2.3x2mm_P0.5mm
- U42: footprint TO_SOT_Packages_SMD:SOT-23-5 -> Package_TO_SOT_SMD:SOT-23-5
- U43: footprint Housings_DFN_QFN:QFN-24-1EP_4x4mm_Pitch0.5mm -> Package_DFN_QFN:QFN-24-1EP_4x4mm_P0.5mm_EP2.7x2.6mm
- renumbered U45 to U44, U44 to U45
Connections:
- wire segments 550 -> 564
Other:
- note added: "VDDA Filter"
- moved on the sheet: C40, C49, C50, C51, C52, C53, C54, C55, D40, D41, D42, D43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

Commit message: changed 3V3 regulator to different IC D20 smaller added 5V RPi Reg EN pulldown
Parts:
- C52, C54: value 10µ -> 22µ
Changed lines of the file:
@@
 P 12250 8625
 F 0 "C54" H 12275 8700 50  0000 L CNN
-F 1 "10µ" H 12275 8550 50  0000 L CNN
+F 1 "22µ" H 12275 8550 50  0000 L CNN
 F 2 "Capacitor_SMD:C_0603_1608Metric" H 12288 8475 50  0001 C CNN
 F 3 "" H 12250 8625 50  0001 C CNN
@@
 P 12250 7500
 F 0 "C52" H 12275 7575 50  0000 L CNN
-F 1 "10µ" H 12275 7425 50  0000 L CNN
+F 1 "22µ" H 12275 7425 50  0000 L CNN
 F 2 "Capacitor_SMD:C_0603_1608Metric" H 12288 7350 50  0001 C CNN
 F 3 "" H 12250 7500 50  0001 C CNN

Commit message: Updated documentation and other small changes
Parts:
- C40: value 1µ -> 2µ2
- C49: value 2µ2 -> 100n
- L40: value 39n -> 1µ
- R40, R41, R43, R44, R45, R46, R52, R53, R54: value 1k6 -> 1k8
- U46: value Buzzer -> Speaker
Connections:
- net LED_4 is gone; now on net LED_3: J40.38 (GPIO20), R50.1
- net LED_1: now also R48.1, U40.96 (PB9); no longer R47.1, U40.95 (PB8)
- net LED_2: now also J40.40 (GPIO21), R49.1; no longer R48.1, U40.96 (PB9)
- net LED_3: no longer J40.40 (GPIO21), R49.1
- new net LED_0: R47.1, U40.95 (PB8)
Changed lines of the file:
@@
 P 9475 1675
 F 0 "U46" H 9675 1725 60  0000 C CNN
-F 1 "Buzzer" H 9750 1650 60  0000 C CNN
+F 1 "Speaker" H 9750 1650 60  0000 C CNN
 F 2 "hedgehog_footprints:Buzzer" H 9475 1675 60  0001 C CNN
 F 3 "" H 9475 1675 60  0001 C CNN
@@
 P 7350 9900
 F 0 "R41" H 7400 9925 50  0000 L CNN
-F 1 "1k6" H 7400 9850 50  0000 L CNN
+F 1 "1k8" H 7400 9850 50  0000 L CNN
 F 2 "Resistor_SMD:R_0603_1608Metric" V 7280 9900 50  0001 C CNN
 F 3 "" H 7350 9900 50  0001 C CNN
@@
 P 4000 6525
 F 0 "R40" H 3800 6575 50  0000 L CNN
-F 1 "1k6" H 3800 6475 50  0000 L CNN
+F 1 "1k8" H 3800 6475 50  0000 L CNN
 F 2 "Resistor_SMD:R_0603_1608Metric" V 3930 6525 50  0001 C CNN
 F 3 "" H 4000 6525 50  0001 C CNN
@@
 P 1875 1800
 F 0 "C40" H 1975 1850 50  0000 L CNN
-F 1 "1µ" H 2000 1775 50  0000 L CNN
+F 1 "2µ2" H 2000 1775 50  0000 L CNN
 F 2 "Capacitor_SMD:C_0603_1608Metric" H 1913 1650 50  0001 C CNN
 F 3 "" H 1875 1800 50  0001 C CNN
@@
 P 1675 1575
 F 0 "L40" V 1750 1575 50  0000 C CNN
-F 1 "39n" V 1625 1575 50  0000 C CNN
+F 1 "1µ" V 1625 1575 50  0000 C CNN
 F 2 "Inductor_SMD:L_0603_1608Metric" H 1675 1575 50  0001 C CNN
 F 3 "" H 1675 1575 50  0001 C CNN
@@
 RPi_UART_TxD
 Text Label 2875 5125 0    60   ~ 0
+LED_0
+Text Label 2875 5225 0    60   ~ 0
 LED_1
-Text Label 2875 5225 0    60   ~ 0
-LED_2
 Text Label 12300 1575 2    60   ~ 0
+LED_0
+Text Label 12300 1775 2    60   ~ 0
 LED_1
-Text Label 12300 1775 2    60   ~ 0
-LED_2
 $Comp
 L Device:R R50
@@
 $EndComp
 Text Label 12300 2000 2    60   ~ 0
+LED_2
+Text Label 12300 2200 2    60   ~ 0
 LED_3
-Text Label 12300 2200 2    60   ~ 0
-LED_4
 Text Label 4200 10275 2    60   ~ 0
-LED_4
+LED_3
 Text Label 4200 10375 2    60   ~ 0
-LED_3
+LED_2
 Text Label 1250 9975 0    60   ~ 0
 STM_BOOT0
@@
 P 8700 9975
 F 0 "C49" H 8725 9900 50  0000 L CNN
-F 1 "2µ2" H 8725 10075 50  0000 L CNN
+F 1 "100n" H 8725 10075 50  0000 L CNN
 F 2 "Capacitor_SMD:C_0603_1608Metric" H 8738 9825 50  0001 C CNN
 F 3 "" H 8700 9975 50  0001 C CNN
@@
 P 9750 4700
 F 0 "R46" H 9625 4650 50  0000 C CNN
-F 1 "1k6" H 9625 4725 50  0000 C CNN
+F 1 "1k8" H 9625 4725 50  0000 C CNN
 F 2 "Resistor_SMD:R_0603_1608Metric" V 9680 4700 50  0001 C CNN
 F 3 "" H 9750 4700 50  0001 C CNN
@@
 P 9650 4700
 F 0 "R45" H 9775 4650 50  0000 C CNN
-F 1 "1k6" H 9775 4725 50  0000 C CNN
+F 1 "1k8" H 9775 4725 50  0000 C CNN
 F 2 "Resistor_SMD:R_0603_1608Metric" V 9580 4700 50  0001 C CNN
 F 3 "" H 9650 4700 50  0001 C CNN
@@
 P 6050 8900
 F 0 "R43" V 5975 8725 50  0000 L CNN
-F 1 "1k6" V 5975 8925 50  0000 L CNN
+F 1 "1k8" V 5975 8925 50  0000 L CNN
 F 2 "Resistor_SMD:R_0603_1608Metric" V 5980 8900 50  0001 C CNN
 F 3 "" H 6050 8900 50  0001 C CNN
@@
 P 5250 10200
 F 0 "R44" H 5300 10225 50  0000 L CNN
-F 1 "1k6" H 5300 10150 50  0000 L CNN
+F 1 "1k8" H 5300 10150 50  0000 L CNN
 F 2 "Resistor_SMD:R_0603_1608Metric" V 5180 10200 50  0001 C CNN
 F 3 "" H 5250 10200 50  0001 C CNN
@@
 P 5825 8350
 F 0 "R52" V 5750 8175 50  0000 L CNN
-F 1 "1k6" V 5750 8375 50  0000 L CNN
+F 1 "1k8" V 5750 8375 50  0000 L CNN
 F 2 "Resistor_SMD:R_0603_1608Metric" V 5755 8350 50  0001 C CNN
 F 3 "" H 5825 8350 50  0001 C CNN
@@
 P 5850 9275
 F 0 "R53" V 5775 9100 50  0000 L CNN
-F 1 "1k6" V 5775 9300 50  0000 L CNN
+F 1 "1k8" V 5775 9300 50  0000 L CNN
 F 2 "Resistor_SMD:R_0603_1608Metric" V 5780 9275 50  0001 C CNN
 F 3 "" H 5850 9275 50  0001 C CNN
@@
 P 5800 10475
 F 0 "R54" V 5725 10300 50  0000 L CNN
-F 1 "1k6" V 5725 10500 50  0000 L CNN
+F 1 "1k8" V 5725 10500 50  0000 L CNN
 F 2 "Resistor_SMD:R_0603_1608Metric" V 5730 10475 50  0001 C CNN
 F 3 "" H 5800 10475 50  0001 C CNN

Commit message: changes for first production version v1.0: added bootstrap resistor R26 R54 Pullup 5V MS Zones bigger U10 Pin7 GND silk improvements version changed: silk, sch & pcb pages updated doc files
Parts:
- D40, D51: value LED -> Red
- D41: value LED -> Yellow
- D42: value LED -> Green
- D43: value LED -> Blue
- J40: value RaspberryPi3 -> Raspberry Pi
Connections:
- net +3V3: now also R54.2
- net GND: no longer R54.2
Other:
- moved on the sheet: R54
Changed lines of the file:
@@
 Sheet 4 5
 Title "Hedgehog"
-Date ""
-Rev "0.4"
+Date "2019-05-12"
+Rev "1.0"
 Comp ""
 Comment1 ""
@@
 P 2725 9375
 F 0 "J40" H 2725 10425 60  0000 C CNN
-F 1 "RaspberryPi3" H 2725 8200 60  0000 C CNN
+F 1 "Raspberry Pi" H 2725 8200 60  0000 C CNN
 F 2 "hedgehog_footprints:Socket_Strip_Straight_2x20_Pitch2.54mm_thermals" H 2725 8350 60  0001 C CNN
 F 3 "" H 2725 8350 60  0001 C CNN
@@
 P 11400 1775
 F 0 "D41" H 11400 1875 50  0000 C CNN
-F 1 "LED" H 11550 1725 50  0000 C CNN
+F 1 "Yellow" H 11600 1725 50  0000 C CNN
 F 2 "LED_SMD:LED_0805_2012Metric" H 11400 1775 50  0001 C CNN
 F 3 "" H 11400 1775 50  0001 C CNN
@@
 P 11400 1575
 F 0 "D40" H 11400 1675 50  0000 C CNN
-F 1 "LED" H 11550 1525 50  0000 C CNN
+F 1 "Red" H 11550 1525 50  0000 C CNN
 F 2 "LED_SMD:LED_0805_2012Metric" H 11400 1575 50  0001 C CNN
 F 3 "" H 11400 1575 50  0001 C CNN
@@
 P 11400 2200
 F 0 "D43" H 11400 2300 50  0000 C CNN
-F 1 "LED" H 11550 2150 50  0000 C CNN
+F 1 "Blue" H 11550 2150 50  0000 C CNN
 F 2 "LED_SMD:LED_0805_2012Metric" H 11400 2200 50  0001 C CNN
 F 3 "" H 11400 2200 50  0001 C CNN
@@
 P 11400 2000
 F 0 "D42" H 11400 2100 50  0000 C CNN
-F 1 "LED" H 11550 1950 50  0000 C CNN
+F 1 "Green" H 11575 1950 50  0000 C CNN
 F 2 "LED_SMD:LED_0805_2012Metric" H 11400 2000 50  0001 C CNN
 F 3 "" H 11400 2000 50  0001 C CNN
@@
 P 11400 1375
 F 0 "D51" H 11400 1475 50  0000 C CNN
-F 1 "LED" H 11550 1325 50  0000 C CNN
+F 1 "Red" H 11550 1325 50  0000 C CNN
 F 2 "LED_SMD:LED_0805_2012Metric" H 11400 1375 50  0001 C CNN
 F 3 "" H 11400 1375 50  0001 C CNN
@@
 $EndComp
 Wire Wire Line
-	5250 10450 5250 10400
-Wire Wire Line
 	5250 10050 5250 10000
 Wire Wire Line
@@
 L Device:R R54
 U 1 1 5BFEACE9
-P 5800 10475
-F 0 "R54" V 5725 10300 50  0000 L CNN
-F 1 "1k8" V 5725 10500 50  0000 L CNN
-F 2 "Resistor_SMD:R_0603_1608Metric" V 5730 10475 50  0001 C CNN
-F 3 "" H 5800 10475 50  0001 C CNN
-	1    5800 10475
+P 5925 10575
+F 0 "R54" V 5850 10400 50  0000 L CNN
+F 1 "1k8" V 5850 10600 50  0000 L CNN
+F 2 "Resistor_SMD:R_0603_1608Metric" V 5855 10575 50  0001 C CNN
+F 3 "" H 5925 10575 50  0001 C CNN
+	1    5925 10575
 	0    1    1    0
 $EndComp
 Wire Wire Line
-	5950 10475 6150 10475
+	6075 10575 6150 10575
 Wire Wire Line
-	6150 10475 6150 10300
+	6150 10575 6150 10300
 Connection ~ 6150 10300
 Wire Wire Line
 	6150 10300 5450 10300
 Wire Wire Line
-	5650 10475 5400 10475
-Wire Wire Line
-	5400 10475 5400 10400
-Wire Wire Line
-	5400 10400 5250 10400
-Connection ~ 5250 10400
-Wire Wire Line
-	5250 10400 5250 10350
-Wire Wire Line
 	14175 7375 14175 7500
 Wire Wire Line
@@
 Wire Notes Line
 	1000 1250 2200 1250
+Wire Wire Line
+	5250 10350 5250 10450
+$Comp
+L power:+3V3 #PWR?
+U 1 1 5C0839DC
+P 5700 10525
+F 0 "#PWR?" H 5700 10375 50  0001 C CNN
+F 1 "+3V3" H 5675 10675 50  0000 C CNN
+F 2 "" H 5700 10525 50  0001 C CNN
+F 3 "" H 5700 10525 50  0001 C CNN
+	1    5700 10525
+	1    0    0    -1
+$EndComp
+Wire Wire Line
+	5700 10525 5700 10575
+Wire Wire Line
+	5700 10575 5775 10575
 $EndSCHEMATC
