File: Reg_5V_MS.sch (KiCad schematic (older format))
At the start: 11 parts, among them Q10 SI7114, U10 RT7259

Commit message: lots of changes: regulator layout improved bom minimized inner top layer completely gnd UB single pole pullups for use without pi swiched to new kicad version and fp lib motor and servo netanmes fixed added input filtering
Parts:
- added C11, C12: 10µ, Capacitor_SMD:C_0603_1608Metric, symbol Device:C
- added C13: 100n, Capacitor_SMD:C_0603_1608Metric, symbol Device:C
- C10: value 22µ -> 10µ; footprint Capacitors_SMD:C_1210 -> Capacitor_SMD:C_0603_1608Metric
- C14: renamed from C11; footprint Capacitors_SMD:C_0603 -> Capacitor_SMD:C_0603_1608Metric
- C15: renamed from C12; footprint Capacitors_SMD:C_0603 -> Capacitor_SMD:C_0603_1608Metric
- C16: renamed from C13; footprint Capacitors_SMD:C_1206 -> Capacitor_SMD:C_1206_3216Metric
- D10: footprint hedgehog_footprints:SOD123F -> Diode_SMD:D_SOD-123F
- Q10: value SI7114 -> SIS434DN; Manucacturer Number SI7114DN-T1-E3 -> SIS434DN-T1-GE3
- R10: footprint Resistors_SMD:R_0603 -> Resistor_SMD:R_0603_1608Metric
- R11: value 43k -> 180k; footprint Resistors_SMD:R_0603 -> Resistor_SMD:R_0603_1608Metric
- R12: value 8k2 -> 34k; footprint Resistors_SMD:R_0603 -> Resistor_SMD:R_0603_1608Metric
Connections:
- net GND: now also C11.1, C12.1, C13.1
- net VIN: now also C11.2, C12.2, C13.2
Changed lines of the file:
@@
 EESchema Schematic File Version 4
 LIBS:Hedgehog-cache
-EELAYER 26 0
+EELAYER 29 0
 EELAYER END
 $Descr A4 11693 8268
 encoding utf-8
 Sheet 2 5
-Title ""
+Title "Hedgehog"
 Date ""
-Rev ""
+Rev "0.4"
 Comp ""
 Comment1 ""
@@
 Comment4 ""
 $EndDescr
-Text HLabel 4050 3200 0    60   Input ~ 0
+Text HLabel 3125 3200 0    60   Input ~ 0
 VIN
 Text HLabel 7975 3350 2    60   Output ~ 0
@@
 $EndComp
 $Comp
-L Device:C C10
-U 1 1 5907CE70
-P 4175 3725
-F 0 "C10" H 4425 3675 50  0000 R CNN
-F 1 "22µ" H 4425 3750 50  0000 R CNN
-F 2 "Capacitors_SMD:C_1210" H 4213 3575 50  0001 C CNN
-F 3 "" H 4175 3725 50  0001 C CNN
-	1    4175 3725
-	-1   0    0    1
-$EndComp
-$Comp
-L Device:C C13
+L Device:C C16
 U 1 1 5907D42E
 P 7425 3825
-F 0 "C13" H 7310 3779 50  0000 R CNN
+F 0 "C16" H 7310 3779 50  0000 R CNN
 F 1 "100µ" H 7310 3870 50  0000 R CNN
-F 2 "Capacitors_SMD:C_1206" H 7463 3675 50  0001 C CNN
+F 2 "Capacitor_SMD:C_1206_3216Metric" H 7463 3675 50  0001 C CNN
 F 3 "" H 7425 3825 50  0001 C CNN
 	1    7425 3825
@@
 F 0 "R10" H 4625 4150 50  0000 L CNN
 F 1 "12k" H 4625 4075 50  0000 L CNN
-F 2 "Resistors_SMD:R_0603" V 4755 4100 50  0001 C CNN
+F 2 "Resistor_SMD:R_0603_1608Metric" V 4755 4100 50  0001 C CNN
 F 3 "" H 4825 4100 50  0001 C CNN
 	1    4825 4100
@@
 $EndComp
 $Comp
-L Device:C C11
+L Device:C C14
 U 1 1 5907D610
 P 4525 3725
-F 0 "C11" H 4775 3675 50  0000 R CNN
+F 0 "C14" H 4775 3675 50  0000 R CNN
 F 1 "1µ" H 4750 3750 50  0000 R CNN
-F 2 "Capacitors_SMD:C_0603" H 4563 3575 50  0001 C CNN
+F 2 "Capacitor_SMD:C_0603_1608Metric" H 4563 3575 50  0001 C CNN
 F 3 "" H 4525 3725 50  0001 C CNN
 	1    4525 3725
@@
 P 7075 3550
 F 0 "R11" H 7145 3596 50  0000 L CNN
-F 1 "43k" H 7145 3505 50  0000 L CNN
-F 2 "Resistors_SMD:R_0603" V 7005 3550 50  0001 C CNN
+F 1 "180k" H 7145 3505 50  0000 L CNN
+F 2 "Resistor_SMD:R_0603_1608Metric" V 7005 3550 50  0001 C CNN
 F 3 "" H 7075 3550 50  0001 C CNN
 	1    7075 3550
@@
 P 7075 4075
 F 0 "R12" H 7145 4121 50  0000 L CNN
-F 1 "8k2" H 7145 4030 50  0000 L CNN
-F 2 "Resistors_SMD:R_0603" V 7005 4075 50  0001 C CNN
+F 1 "34k" H 7145 4030 50  0000 L CNN
+F 2 "Resistor_SMD:R_0603_1608Metric" V 7005 4075 50  0001 C CNN
 F 3 "" H 7075 4075 50  0001 C CNN
 	1    7075 4075
@@
 F 0 "D10" V 7779 3904 50  0000 L CNN
 F 1 "5.2V" V 7870 3904 50  0000 L CNN
-F 2 "hedgehog_footprints:SOD123F" H 7825 3825 50  0001 C CNN
+F 2 "Diode_SMD:D_SOD-123F" H 7825 3825 50  0001 C CNN
 F 3 "" H 7825 3825 50  0001 C CNN
 F 4 "NZH5V1B,115" V 7825 3825 60  0001 C CNN "Manufacturer Code"
@@
 $EndComp
 $Comp
-L Device:C C12
+L Device:C C15
 U 1 1 5907D2A6
 P 6175 3200
-F 0 "C12" V 6375 3200 50  0000 C CNN
+F 0 "C15" V 6375 3200 50  0000 C CNN
 F 1 "1µ" V 6300 3200 50  0000 C CNN
-F 2 "Capacitors_SMD:C_0603" H 6213 3050 50  0001 C CNN
+F 2 "Capacitor_SMD:C_0603_1608Metric" H 6213 3050 50  0001 C CNN
 F 3 "" H 6175 3200 50  0001 C CNN
 	1    6175 3200
@@
 	4975 3750 4875 3750
 Wire Wire Line
-	4975 3850 4750 3850
+	4975 3850 4825 3850
 Wire Wire Line
 	4825 3850 4825 3950
@@
 	5525 4325 5525 4300
 Wire Wire Line
-	4175 4325 7825 4325
+	4175 4325 4525 4325
 Wire Wire Line
 	5425 4325 5425 4300
@@
 	4525 3550 4525 3575
 Wire Wire Line
-	4050 3200 4975 3200
-Wire Wire Line
-	4925 3200 4925 3400
+	3125 3200 3500 3200
+Wire Wire Line
+	4925 3200 4925 3300
 Wire Wire Line
 	4925 3400 4975 3400
@@
 P 6325 3750
 F 0 "Q10" H 6530 3796 50  0000 L CNN
-F 1 "SI7114" H 6530 3705 50  0000 L CNN
+F 1 "SIS434DN" H 6530 3705 50  0000 L CNN
 F 2 "hedgehog_footprints:PowerPAK_1212-8" H 6525 3850 50  0001 C CNN
 F 3 "" H 6325 3750 50  0001 C CNN
-F 4 "SI7114DN-T1-E3" H 6325 3750 60  0001 C CNN "Manucacturer Number"
+F 4 "SIS434DN-T1-GE3" H 6325 3750 60  0001 C CNN "Manucacturer Number"
 	1    6325 3750
 	1    0    0    -1
@@
 	5975 3550 6025 3550
 Wire Wire Line
-	6025 3550 6025 3350
-Wire Wire Line
-	5975 3350 6625 3350
+	6025 3550 6025 3450
+Wire Wire Line
+	5975 3350 6025 3350
 Wire Wire Line
 	5975 3450 6025 3450
@@
 Connection ~ 6425 3350
 Wire Wire Line
-	6925 3350 7975 3350
+	6925 3350 7075 3350
 Wire Wire Line
 	7825 3350 7825 3675
@@
 Connection ~ 7075 3350
 Wire Wire Line
-	7075 3700 7075 3925
+	7075 3700 7075 3850
 Wire Wire Line
 	7075 4225 7075 4325
@@
 	1    0    0    -1
 $EndComp
+Wire Wire Line
+	4825 3850 4750 3850
+Wire Wire Line
+	5475 4325 5525 4325
+Wire Wire Line
+	5425 4325 5475 4325
+Wire Wire Line
+	4825 4325 5425 4325
+Wire Wire Line
+	4525 4325 4825 4325
+Wire Wire Line
+	4925 3300 4925 3400
+Wire Wire Line
+	4925 3200 4975 3200
+Wire Wire Line
+	5525 4325 6425 4325
+Wire Wire Line
+	6025 3450 6025 3350
+Wire Wire Line
+	6025 3350 6325 3350
+Wire Wire Line
+	6325 3350 6425 3350
+Wire Wire Line
+	6425 3350 6625 3350
+Wire Wire Line
+	7825 3350 7975 3350
+Wire Wire Line
+	6425 4325 7075 4325
+Wire Wire Line
+	7075 3350 7425 3350
+Wire Wire Line
+	7075 4325 7425 4325
+Wire Wire Line
+	7075 3850 7075 3925
+Wire Wire Line
+	7425 3350 7825 3350
+Wire Wire Line
+	7425 4325 7825 4325
+Wire Wire Line
+	4175 3200 4925 3200
+$Comp
+L Device:C C13
+U 1 1 5A9C895D
+P 4175 3725
+F 0 "C13" H 4325 3550 50  0000 R CNN
+F 1 "100n" H 4375 3625 50  0000 R CNN
+F 2 "Capacitor_SMD:C_0603_1608Metric" H 4213 3575 50  0001 C CNN
+F 3 "" H 4175 3725 50  0001 C CNN
+	1    4175 3725
+	-1   0    0    1
+$EndComp
+$Comp
+L Device:C C12
+U 1 1 5A9C8A69
+P 3950 3725
+F 0 "C12" H 4100 3550 50  0000 R CNN
+F 1 "10µ" H 4125 3625 50  0000 R CNN
+F 2 "Capacitor_SMD:C_0603_1608Metric" H 3988 3575 50  0001 C CNN
+F 3 "" H 3950 3725 50  0001 C CNN
+	1    3950 3725
+	-1   0    0    1
+$EndComp
+$Comp
+L Device:C C11
+U 1 1 5A9CCC4E
+P 3725 3725
+F 0 "C11" H 3875 3550 50  0000 R CNN
+F 1 "10µ" H 3900 3625 50  0000 R CNN
+F 2 "Capacitor_SMD:C_0603_1608Metric" H 3763 3575 50  0001 C CNN
+F 3 "" H 3725 3725 50  0001 C CNN
+	1    3725 3725
+	-1   0    0    1
+$EndComp
+$Comp
+L Device:C C10
+U 1 1 5A9CCC96
+P 3500 3725
+F 0 "C10" H 3650 3550 50  0000 R CNN
+F 1 "10µ" H 3675 3625 50  0000 R CNN
+F 2 "Capacitor_SMD:C_0603_1608Metric" H 3538 3575 50  0001 C CNN
+F 3 "" H 3500 3725 50  0001 C CNN
+	1    3500 3725
+	-1   0    0    1
+$EndComp
+Wire Wire Line
+	4175 4325 3950 4325
+Wire Wire Line
+	3500 4325 3500 3875
+Connection ~ 4175 4325
+Wire Wire Line
+	3725 3875 3725 4325
+Connection ~ 3725 4325
+Wire Wire Line
+	3725 4325 3500 4325
+Wire Wire Line
+	3950 3875 3950 4325
+Connection ~ 3950 4325
+Wire Wire Line
+	3950 4325 3725 4325
+Wire Wire Line
+	3950 3575 3950 3200
+Connection ~ 3950 3200
+Wire Wire Line
+	3950 3200 4175 3200
+Wire Wire Line
+	3725 3575 3725 3200
+Connection ~ 3725 3200
+Wire Wire Line
+	3725 3200 3950 3200
+Wire Wire Line
+	3500 3575 3500 3200
+Connection ~ 3500 3200
+Wire Wire Line
+	3500 3200 3725 3200
 $EndSCHEMATC

Commit message: Updated documentation and other small changes
Parts:
- Q10: value SIS434DN -> SIS488DN
- R10: value 12k -> 1k8
Changed lines of the file:
@@
 P 4825 4100
 F 0 "R10" H 4625 4150 50  0000 L CNN
-F 1 "12k" H 4625 4075 50  0000 L CNN
+F 1 "1k8" H 4625 4075 50  0000 L CNN
 F 2 "Resistor_SMD:R_0603_1608Metric" V 4755 4100 50  0001 C CNN
 F 3 "" H 4825 4100 50  0001 C CNN
@@
 P 6325 3750
 F 0 "Q10" H 6530 3796 50  0000 L CNN
-F 1 "SIS434DN" H 6530 3705 50  0000 L CNN
+F 1 "SIS488DN" H 6530 3705 50  0000 L CNN
 F 2 "hedgehog_footprints:PowerPAK_1212-8" H 6525 3850 50  0001 C CNN
 F 3 "" H 6325 3750 50  0001 C CNN

Commit message: changes for first production version v1.0: added bootstrap resistor R26 R54 Pullup 5V MS Zones bigger U10 Pin7 GND silk improvements version changed: silk, sch & pcb pages updated doc files
Connections:
- net GND: now also U10.7 (NC)
Changed lines of the file:
@@
 Sheet 2 5
 Title "Hedgehog"
-Date ""
-Rev "0.4"
+Date "2019-05-12"
+Rev "1.0"
 Comp ""
 Comment1 ""
@@
 	5425 4325 5475 4325
 Wire Wire Line
-	4825 4325 5425 4325
+	4825 4325 4975 4325
 Wire Wire Line
 	4525 4325 4825 4325
@@
 Wire Wire Line
 	3500 3200 3725 3200
+Wire Wire Line
+	4975 4000 4975 4325
+Connection ~ 4975 4325
+Wire Wire Line
+	4975 4325 5425 4325
 $EndSCHEMATC
